Commit message: Move generated Robot Digital Twin URDF assets

File: assets/generated_urdf/robot_digital_twin/camera.urdf (robot description, URDF)
Before this commit: robot camera, 4 links, 3 joints
Links:
- link link_camera: geometry collision mesh filename=../../../third_party/Robot_Digital_Twin/gazebo/meshes/eoat/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; visual mesh filename=../../../third_party/Robot_Digital_Twin/gazebo/meshes/eoat/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

File: assets/generated_urdf/robot_digital_twin/dual_gp4.urdf (robot description, URDF)
Before this commit: robot dual_gp4, 24 links, 23 joints
Links:
- link left_arm_base_link: geometry collision mesh filename=../../../third_party/Robot_Digital_Twin/gazebo/meshes/gp4/b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; visual mesh filename=../../../third_party/Robot_Digital_Twin/gazebo/meshes/gp4/b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
- link left_arm_link_1: geometry collision mesh filename=../../../third_party/Robot_Digital_Twin/gazebo/meshes/gp4/l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; visual mesh filename=../../../third_party/Robot_Digital_Twin/gazebo/meshes/gp4/l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
- link left_arm_link_2: geometry collision mesh filename=../../../third_party/Robot_Digital_Twin/gazebo/meshes/gp4/l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; visual mesh filename=../../../third_party/Robot_Digital_Twin/gazebo/meshes/gp4/l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
- link left_arm_link_3: geometry collision mesh filename=../../../third_party/Robot_Digital_Twin/gazebo/meshes/gp4/l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; visual mesh filename=../../../third_party/Robot_Digital_Twin/gazebo/meshes/gp4/l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
- link left_arm_link_4: geometry collision mesh filename=../../../third_party/Robot_Digital_Twin/gazebo/meshes/gp4/l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; visual mesh filename=../../../third_party/Robot_Digital_Twin/gazebo/meshes/gp4/l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
- link left_arm_link_5: geometry collision mesh filename=../../../third_party/Robot_Digital_Twin/gazebo/meshes/gp4/l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; visual mesh filename=../../../third_party/Robot_Digital_Twin/gazebo/meshes/gp4/l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
- link left_arm_link_6: geometry collision mesh filename=../../../third_party/Robot_Digital_Twin/gazebo/meshes/gp4/l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; visual mesh filename=../../../third_party/Robot_Digital_Twin/gazebo/meshes/gp4/l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
- link left_arm_link_tool: geometry collision mesh filename=../../../third_party/Robot_Digital_Twin/gazebo/meshes/eoat/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; visual mesh filename=../../../third_party/Robot_Digital_Twin/gazebo/meshes/eoat/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
- link right_arm_base_link: geometry collision mesh filename=../../../third_party/Robot_Digital_Twin/gazebo/meshes/gp4/b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; visual mesh filename=../../../third_party/Robot_Digital_Twin/gazebo/meshes/gp4/b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
- link right_arm_link_1: geometry collision mesh filename=../../../third_party/Robot_Digital_Twin/gazebo/meshes/gp4/l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; visual mesh filename=../../../third_party/Robot_Digital_Twin/gazebo/meshes/gp4/l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
- link right_arm_link_2: geometry collision mesh filename=../../../third_party/Robot_Digital_Twin/gazebo/meshes/gp4/l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; visual mesh filename=../../../third_party/Robot_Digital_Twin/gazebo/meshes/gp4/l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
- link right_arm_link_3: geometry collision mesh filename=../../../third_party/Robot_Digital_Twin/gazebo/meshes/gp4/l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; visual mesh filename=../../../third_party/Robot_Digital_Twin/gazebo/meshes/gp4/l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
- link right_arm_link_4: geometry collision mesh filename=../../../third_party/Robot_Digital_Twin/gazebo/meshes/gp4/l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; visual mesh filename=../../../third_party/Robot_Digital_Twin/gazebo/meshes/gp4/l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
- link right_arm_link_5: geometry collision mesh filename=../../../third_party/Robot_Digital_Twin/gazebo/meshes/gp4/l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; visual mesh filename=../../../third_party/Robot_Digital_Twin/gazebo/meshes/gp4/l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
- link right_arm_link_6: geometry collision mesh filename=../../../third_party/Robot_Digital_Twin/gazebo/meshes/gp4/l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; visual mesh filename=../../../third_party/Robot_Digital_Twin/gazebo/meshes/gp4/l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
- link right_arm_link_tool: geometry collision mesh filename=../../../third_party/Robot_Digital_Twin/gazebo/meshes/eoat/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; visual mesh filename=../../../third_party/Robot_Digital_Twin/gazebo/meshes/eoat/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
Joints:
- removed joint left_arm_to_${connected_to}
- removed joint right_arm_to_${connected_to}
- added joint left_arm_to_base: type fixed, parent base, child left_arm_base, origin xyz=0 0 0.9246 rpy=0 0 0
- added joint right_arm_to_base: type fixed, parent base, child right_arm_base, origin xyz=0.88101137 -0.01304334 0.92460000 rpy=0 0 3.13585279
- joint left_arm_joint_1: limit lower=${radians(-170)} upper=${radians(170)} effort=0 velocity=${radians(465)} -> lower=-2.96705972839 upper=2.96705972839 effort=0 velocity=8.11578102177
- joint left_arm_joint_2: limit lower=${radians(-110)} upper=${radians(130)} effort=100 velocity=${radians(465)} -> lower=-1.91986217719 upper=2.26892802759 effort=100 velocity=8.11578102177
- joint left_arm_joint_3: limit lower=${radians(-65)} upper=${radians(200)} effort=0 velocity=${radians(525)} -> lower=-1.1344640138 upper=3.49065850399 effort=0 velocity=9.16297857297
- joint left_arm_joint_4: limit lower=${radians(-200)} upper=${radians(200)} effort=0 velocity=${radians(550)} -> lower=-3.49065850399 upper=3.49065850399 effort=0 velocity=9.59931088597
- joint left_arm_joint_5: limit lower=${radians(-123)} upper=${radians(123)} effort=0 velocity=${radians(545)} -> lower=-2.14675497995 upper=2.14675497995 effort=0 velocity=9.51204442337
- joint left_arm_joint_6: limit lower=${radians(-455)} upper=${radians(455)} effort=0 velocity=${radians(1000)} -> lower=-7.94124809657 upper=7.94124809657 effort=0 velocity=17.4532925199
- joint right_arm_joint_1: limit lower=${radians(-170)} upper=${radians(170)} effort=0 velocity=${radians(465)} -> lower=-2.96705972839 upper=2.96705972839 effort=0 velocity=8.11578102177
- joint right_arm_joint_2: limit lower=${radians(-110)} upper=${radians(130)} effort=100 velocity=${radians(465)} -> lower=-1.91986217719 upper=2.26892802759 effort=100 velocity=8.11578102177
- joint right_arm_joint_3: limit lower=${radians(-65)} upper=${radians(200)} effort=0 velocity=${radians(525)} -> lower=-1.1344640138 upper=3.49065850399 effort=0 velocity=9.16297857297
- joint right_arm_joint_4: limit lower=${radians(-200)} upper=${radians(200)} effort=0 velocity=${radians(550)} -> lower=-3.49065850399 upper=3.49065850399 effort=0 velocity=9.59931088597
- joint right_arm_joint_5: limit lower=${radians(-123)} upper=${radians(123)} effort=0 velocity=${radians(545)} -> lower=-2.14675497995 upper=2.14675497995 effort=0 velocity=9.51204442337
- joint right_arm_joint_6: limit lower=${radians(-455)} upper=${radians(455)} effort=0 velocity=${radians(1000)} -> lower=-7.94124809657 upper=7.94124809657 effort=0 velocity=17.4532925199

File: assets/generated_urdf/robot_digital_twin/env.urdf (robot description, URDF)
Before this commit: robot testbed_env, 3 links, 2 joints
Links:
- link env: geometry visual mesh filename=../../../third_party/Robot_Digital_Twin/gazebo/meshes/env/t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

File: assets/generated_urdf/robot_digital_twin/fanuc_arm.urdf (robot description, URDF)
Before this commit: robot Yaskawa_gp4, 12 links, 11 joints
Links:
- removed link flange
- added link link_camera, mass 0.10811; collision mesh filename=../../../third_party/Robot_Digital_Twin/gazebo/meshes/eoat/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; visual mesh filename=../../../third_party/Robot_Digital_Twin/gazebo/meshes/eoat/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
- added link link_camera_origin, mass 1e-5; collision box size=0.0001 0.0001 0.0001; visual box size=0.0001 0.01 0.01
- added link link_precam, mass 1e-5
- link base_link: geometry collision mesh filename=../../../third_party/Robot_Digital_Twin/gazebo/meshes/lrmat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; visual mesh filename=../../../third_party/Robot_Digital_Twin/gazebo/meshes/lrmat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
- link fts: geometry collision cylinder length=0.041 radius=0.035; visual cylinder length=0.041 radius=0.035
- link link_1: geometry collision mesh filename=../../../third_party/Robot_Digital_Twin/gazebo/meshes/lrmat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; visual mesh filename=../../../third_party/Robot_Digital_Twin/gazebo/meshes/lrmat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
- link link_2: geometry collision mesh filename=../../../third_party/Robot_Digital_Twin/gazebo/meshes/lrmat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; visual mesh filename=../../../third_party/Robot_Digital_Twin/gazebo/meshes/lrmat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
- link link_3: geometry collision mesh filename=../../../third_party/Robot_Digital_Twin/gazebo/meshes/lrmat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; visual mesh filename=../../../third_party/Robot_Digital_Twin/gazebo/meshes/lrmat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
- link link_4: geometry collision mesh filename=../../../third_party/Robot_Digital_Twin/gazebo/meshes/lrmat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; visual mesh filename=../../../third_party/Robot_Digital_Twin/gazebo/meshes/lrmat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
- link link_5: geometry collision mesh filename=../../../third_party/Robot_Digital_Twin/gazebo/meshes/lrmat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; visual mesh filename=../../../third_party/Robot_Digital_Twin/gazebo/meshes/lrmat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
- link link_6: geometry collision mesh filename=../../../third_party/Robot_Digital_Twin/gazebo/meshes/lrmat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; visual mesh filename=../../../third_party/Robot_Digital_Twin/gazebo/meshes/lrmat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
- link link_tool: geometry visual mesh filename=../../../third_party/Robot_Digital_Twin/gazebo/meshes/eoat/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
Joints:
- removed joint joint_6_t-flange
- added joint camera_imgplane: type fixed, parent link_camera, child link_camera_origin, origin xyz=0.013 0.0 0.0305 rpy=0 0 0
- added joint precam_camera: type fixed, parent link_precam, child link_camera, origin xyz=0 0 0 rpy=0 0.785398163397 0
- added joint tool_precam: type fixed, parent link_tool, child link_precam, origin xyz=0 -0.062194148 -0.005909903 rpy=1.57079632679 -1.57079632679  0
- joint fts_tool: origin xyz=0 0 0.02525 rpy=0 0 3.14159265359 -> xyz=0 0 0.02185 rpy=0 0 3.14159265359
- joint joint_2: origin xyz=0 0 0 rpy=0 0 0 -> xyz=0.050 0 0 rpy=0 0 0
- joint joint_3: origin xyz=0 0 0.260 rpy=0 0 0 -> xyz=0 0 0.440 rpy=0 0 0
- joint joint_4: origin xyz=0.290 0 0.015 rpy=0 0 0 -> xyz=0 0 0.035 rpy=0 0 0
- joint joint_5: origin xyz=0 0 0 rpy=0 0 0 -> xyz=0.420 0 0 rpy=0 0 0
- joint joint_6: origin xyz=0 0 0 rpy=0 0 0 -> xyz=0.080 0 0 rpy=0 0 0
- joint link_6_fts: origin xyz=0.02525 0 0 rpy=0 1.57079632679 0 -> xyz=0.02185 0 0 rpy=0 1.57079632679 0; parent flange -> link_6

File: assets/generated_urdf/robot_digital_twin/gp4.urdf (robot description, URDF)
Before this commit: robot Yaskawa_gp50, 9 links, 8 joints
Links:
- added link flange
- added link fts, mass 1e-5; collision cylinder length=0.0505 radius=0.035; visual cylinder length=0.0505 radius=0.035
- added link link_tool, mass 0.10811; visual mesh filename=../../../third_party/Robot_Digital_Twin/gazebo/meshes/eoat/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
- link base_link: geometry collision mesh filename=../../../third_party/Robot_Digital_Twin/gazebo/meshes/gp4/b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; visual mesh filename=../../../third_party/Robot_Digital_Twin/gazebo/meshes/gp4/b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
- link link_1: geometry collision mesh filename=../../../third_party/Robot_Digital_Twin/gazebo/meshes/gp4/l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; visual mesh filename=../../../third_party/Robot_Digital_Twin/gazebo/meshes/gp4/l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
- link link_2: geometry collision mesh filename=../../../third_party/Robot_Digital_Twin/gazebo/meshes/gp4/l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; visual mesh filename=../../../third_party/Robot_Digital_Twin/gazebo/meshes/gp4/l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
- link link_3: geometry collision mesh filename=../../../third_party/Robot_Digital_Twin/gazebo/meshes/gp4/l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; visual mesh filename=../../../third_party/Robot_Digital_Twin/gazebo/meshes/gp4/l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
- link link_4: geometry collision mesh filename=../../../third_party/Robot_Digital_Twin/gazebo/meshes/gp4/l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; visual mesh filename=../../../third_party/Robot_Digital_Twin/gazebo/meshes/gp4/l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
- link link_5: geometry collision mesh filename=../../../third_party/Robot_Digital_Twin/gazebo/meshes/gp4/l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; visual mesh filename=../../../third_party/Robot_Digital_Twin/gazebo/meshes/gp4/l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
- link link_6: geometry collision mesh filename=../../../third_party/Robot_Digital_Twin/gazebo/meshes/gp4/l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; visual mesh filename=../../../third_party/Robot_Digital_Twin/gazebo/meshes/gp4/l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
Joints:
- added joint fts_tool: type revolute, parent fts, child link_tool, origin xyz=0 0 0.02525 rpy=0 0 3.14159265359, axis 0 0 1, limit lower=0 upper=0 effort=0 velocity=0
- added joint joint_6_t-flange: type fixed, parent link_6, child flange, origin xyz=0.072 0 0 rpy=0 0 0
- added joint link_6_fts: type fixed, parent flange, child fts, origin xyz=0.02525 0 0 rpy=0 1.57079632679 0
- joint joint_1: axis 0 1 0 -> 0 0 1; origin xyz=0 0 0.223 rpy=1.5708 0 0 -> xyz=0 0 0.330 rpy=0 0 0
- joint joint_2: axis 0 0 -1 -> 0 1 0; origin xyz=0.145 0.315 0.0435 rpy=0 0 0 -> xyz=0 0 0 rpy=0 0 0
- joint joint_3: axis 0 0 1 -> 0 -1 0; origin xyz=0 0.87 0 rpy=0 0 0 -> xyz=0 0 0.260 rpy=0 0 0
- joint joint_4: origin xyz=0.317 0.21 -0.0435 rpy=0 0 0 -> xyz=0.290 0 0.015 rpy=0 0 0
- joint joint_5: axis 0 0 1 -> 0 -1 0; origin xyz=0.7065 0 0 rpy=0 0 0 -> xyz=0 0 0 rpy=0 0 0
- joint joint_6: axis 0 0 -1 -> -1 0 0; origin xyz=0.174 0 -0.001 rpy=1.5708 0 1.5708 -> xyz=0 0 0 rpy=0 0 0

File: assets/generated_urdf/robot_digital_twin/lego_1x1.urdf (robot description, URDF)
Before this commit: robot b2x6, 1 links, 0 joints
Links:
- link brick: geometry visual mesh filename=../../../third_party/Robot_Digital_Twin/gazebo/meshes/lego/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 scale=0.001 0.001 0.001

File: assets/generated_urdf/robot_digital_twin/lego_1x2.urdf (robot description, URDF)
Before this commit: robot b1x2, 1 links, 0 joints
Links:
- link brick: geometry visual mesh filename=../../../third_party/Robot_Digital_Twin/gazebo/meshes/lego/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 scale=0.001 0.001 0.001

File: assets/generated_urdf/robot_digital_twin/lego_1x4.urdf (robot description, URDF)
Before this commit: robot b2x4, 1 links, 0 joints
Links:
- link brick: geometry visual mesh filename=../../../third_party/Robot_Digital_Twin/gazebo/meshes/lego/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 scale=0.001 0.001 0.001

File: assets/generated_urdf/robot_digital_twin/lego_1x6.urdf (robot description, URDF)
Before this commit: robot base_plate48, 1 links, 0 joints
Links:
- removed link plate
- added link brick, mass 0.001; visual mesh filename=../../../third_party/Robot_Digital_Twin/gazebo/meshes/lego/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 scale=0.001 0.001 0.001

File: assets/generated_urdf/robot_digital_twin/lego_1x8.urdf (robot description, URDF)
Before this commit: robot b2x8, 1 links, 0 joints
Links:
- link brick: geometry visual mesh filename=../../../third_party/Robot_Digital_Twin/gazebo/meshes/lego/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 scale=0.001 0.001 0.001

File: assets/generated_urdf/robot_digital_twin/lego_2x2.urdf (robot description, URDF)
Before this commit: robot b2x2, 1 links, 0 joints
Links:
- link brick: geometry visual mesh filename=../../../third_party/Robot_Digital_Twin/gazebo/meshes/lego/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 scale=0.001 0.001 0.001

File: assets/generated_urdf/robot_digital_twin/lego_2x4.urdf (robot description, URDF)
Before this commit: robot b1x4, 1 links, 0 joints
Links:
- link brick: geometry visual mesh filename=../../../third_party/Robot_Digital_Twin/gazebo/meshes/lego/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 scale=0.001 0.001 0.001

File: assets/generated_urdf/robot_digital_twin/lego_2x6.urdf (robot description, URDF)
Before this commit: robot base_plate, 1 links, 0 joints
Links:
- removed link plate
- added link brick, mass 0.001; visual mesh filename=../../../third_party/Robot_Digital_Twin/gazebo/meshes/lego/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 scale=0.001 0.001 0.001

File: assets/generated_urdf/robot_digital_twin/lego_2x8.urdf (robot description, URDF)
Before this commit: robot b1x8, 1 links, 0 joints
Links:
- link brick: geometry visual mesh filename=../../../third_party/Robot_Digital_Twin/gazebo/meshes/lego/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 scale=0.001 0.001 0.001

File: assets/generated_urdf/robot_digital_twin/lego_baseplate.urdf (robot description, URDF)
Before this commit: robot b1x6, 1 links, 0 joints
Links:
- removed link brick
- added link plate, mass 0.001; visual mesh filename=../../../third_party/Robot_Digital_Twin/gazebo/meshes/lego/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 scale=0.001 0.001 0.001

File: assets/generated_urdf/robot_digital_twin/lego_baseplate32.urdf (robot description, URDF)
Before this commit: robot base_plate32, 1 links, 0 joints
Links:
- link plate: geometry visual mesh filename=../../../third_party/Robot_Digital_Twin/gazebo/meshes/lego/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 scale=0.001 0.001 0.001

File: assets/generated_urdf/robot_digital_twin/lego_baseplate48.urdf (robot description, URDF)
Before this commit: robot b1x1, 1 links, 0 joints
Links:
- removed link brick
- added link plate, mass 0.001; visual mesh filename=../../../third_party/Robot_Digital_Twin/gazebo/meshes/lego/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 scale=0.001 0.001 0.001
