Commit message: Refine RM75 LEGO tool assets and validation docs

File: assets/rm75_gripper/RM75-B/urdf/RM75-B_lego_tool.urdf (robot description, URDF)
Before this commit: robot RM75B_with_LegoTool, 11 links, 10 joints
Links:
- link lego_tool_link: geometry collision mesh filename=../meshes/lego_test_open_fixed.stl scale=0.001 0.001 0.001; visual mesh filename=../meshes/lego_test_open_fixed.stl scale=0.001 0.001 0.001

Commit message: Calibrate RM75 LEGO contact frame and add stage motions

File: assets/rm75_gripper/RM75-B/urdf/RM75-B_lego_tool.urdf (robot description, URDF)
Before this commit: robot RM75B_with_Gripper_LegoTool, 11 links, 10 joints
Joints:
- joint lego_tool_tcp_joint: origin xyz=0 0 0.075000 rpy=0 0 0 -> xyz=-0.001000 0 0.057000 rpy=0 0 0
